Commit message: should fix the gimbal oscillation problem, if not, god bless teamhku

File: urdf/hku_m100_base_with_gimbal.urdf.xacro (robot description, xacro)
@@ -63,5 +63,5 @@
   </xacro:gimbal_camera>
  -->
-   <joint name="camera_joint" type="continuous">
+   <joint name="camera_joint" type="floating">
       <origin xyz="0.1 0 -0.04" rpy="0 0 0"/>
       <parent link="base_link"/>
@@ -87,5 +87,5 @@
       </collision>
     </link>
-    <joint name="camera_optical_joint" type="fixed">
+    <joint name="camera_optical_joint" type="continuous">
       <origin xyz="0 0 0" rpy="${-M_PI/2} 0.0 ${-M_PI/2}" />
       <parent link="camera_link" />

Commit message: fix the gimbal orientation bug

File: urdf/hku_m100_base_with_gimbal.urdf.xacro (robot description, xacro)
@@ -87,5 +87,5 @@
       </collision>
     </link>
-    <joint name="camera_optical_joint" type="continuous">
+    <joint name="camera_optical_joint" type="floating">
       <origin xyz="0 0 0" rpy="${-M_PI/2} 0.0 ${-M_PI/2}" />
       <parent link="camera_link" />
@@ -98,5 +98,6 @@
         <camera>
           <!-- <pose>0.027 0 -0.027 0 1.57 0</pose> -->
-          <pose>0.027 0 -0.027 0 1.57 0</pose>
+          <!-- <pose>0.027 0 -0.027 0 1.57 0</pose> -->
+          <pose>0.027 0 -0.027 0 0 0</pose>
           <horizontal_fov>${94 * M_PI/180.0}</horizontal_fov>
           <image>
